File: Kicad/Custom Keyboard.kicad_pcb (KiCad board)
At the start: 2 copper layers, 349.3 x 133.3 mm, 216 parts, among them SW1 SW_Push, SW10 SW_Push, SW11 SW_Push, SW12 SW_Push, SW13 SW_Push, SW14 SW_Push, SW15 SW_Push, SW16 SW_Push, SW17 SW_Push, SW18 SW_Push, SW19 SW_Push, SW2 SW_Push, SW20 SW_Push, SW21 SW_Push, SW22 SW_Push, SW23 SW_Push, SW24 SW_Push, SW25 SW_Push, SW26 SW_Push, SW27 SW_Push, SW28 SW_Push, SW29 SW_Push, SW3 SW_Push, SW30 SW_Push, SW31 SW_Push, SW32 SW_Push, SW33 SW_Push, SW34 SW_Push, SW35 SW_Push, SW36 SW_Push, SW37 SW_Push, SW38 SW_Push, SW39 SW_Push, SW4 SW_Push, SW40 SW_Push, SW41 SW_Push, SW42 SW_Push, SW43 SW_Push, SW44 SW_Push, SW45 SW_Push, SW46 SW_Push, SW47 SW_Push, SW48 SW_Push, SW49 SW_Push, SW5 SW_Push, SW50 SW_Push, SW51 SW_Push, SW52 SW_Push, SW53 SW_Push, SW54 SW_Push, SW55 SW_Push, SW56 SW_Push, SW57 SW_Push, SW58 SW_Push, SW59 SW_Push, SW6 SW_Push, SW60 SW_Push, SW61 SW_Push, SW62 SW_Push, SW63 SW_Push, SW64 SW_Push, SW65 SW_Push, SW66 SW_Push, SW7 SW_Push, SW8 SW_Push, SW9 SW_Push, U1 ER_OLEDM0.91_1x-I2C, U4 PCF8574AP

Commit message: replacing fabs
Parts:
- added C2: 0.1uF, Capacitor_THT:C_Disc_D5.0mm_W2.5mm_P5.00mm, F.Cu at (429.6, 163.0)
- added C3: 0.1uF, Capacitor_THT:C_Disc_D5.0mm_W2.5mm_P5.00mm, F.Cu at (480.3, 252.6)
- C1: footprint Capacitor_THT:CP_Radial_D8.0mm_P3.50mm -> Capacitor_THT:CP_Radial_D12.5mm_P5.00mm
- R3: value R -> 4.7k
- U3: value ~ -> SN74AHCT125N
- moved C1 110.3 mm to (210.4, 255.6)
- moved U3 7.32 mm to (468.9, 250.9)
- moved R1 4.44 mm to (465.4, 254.8)
Connections:
- net RGB_Data_Out renamed RGB_Out
Routing:
- net +3V3: track 349.3 -> 363.5 mm
- net +5V: track 2179.3 -> 2189.1 mm, vias 68 -> 70
- net /RGB Data: track 96.5 -> 87.1 mm
- net Net-(RGB_LED1-DIN): track 426.8 -> 433.4 mm
- net RGB_Out: track 6.49 -> 3.64 mm, vias 1 -> 0
