File: Kicad/Custom Keyboard.kicad_sch (KiCad schematic)
At the start: 212 parts, among them SW1 SW_Push, SW10 SW_Push, SW11 SW_Push, SW12 SW_Push, SW13 SW_Push, SW14 SW_Push, SW15 SW_Push, SW16 SW_Push, SW17 SW_Push, SW18 SW_Push, SW19 SW_Push, SW2 SW_Push, SW20 SW_Push, SW21 SW_Push, SW22 SW_Push, SW23 SW_Push, SW24 SW_Push, SW25 SW_Push, SW26 SW_Push, SW27 SW_Push, SW28 SW_Push, SW29 SW_Push, SW3 SW_Push, SW30 SW_Push, SW31 SW_Push, SW32 SW_Push, SW33 SW_Push, SW34 SW_Push, SW35 SW_Push, SW36 SW_Push, SW37 SW_Push, SW38 SW_Push, SW39 SW_Push, SW4 SW_Push, SW40 SW_Push, SW41 SW_Push, SW42 SW_Push, SW43 SW_Push, SW44 SW_Push, SW45 SW_Push, SW46 SW_Push, SW47 SW_Push, SW48 SW_Push, SW49 SW_Push, SW5 SW_Push, SW50 SW_Push, SW51 SW_Push, SW52 SW_Push, SW53 SW_Push, SW54 SW_Push, SW55 SW_Push, SW56 SW_Push, SW57 SW_Push, SW58 SW_Push, SW59 SW_Push, SW6 SW_Push, SW60 SW_Push, SW61 SW_Push, SW62 SW_Push, SW63 SW_Push, SW64 SW_Push, SW65 SW_Push, SW66 SW_Push, SW7 SW_Push, SW8 SW_Push, SW9 SW_Push, U1 ER_OLEDM0.91_1x-I2C, U2 MCP23017x-x-SO

Commit message: Rearranging files
Parts:
- removed U2: MCP23017x-x-SO, Package_SO:SOIC-28W_7.5x17.9mm_P1.27mm, symbol Interface_Expansion:MCP23017x-x-SO
- added R2: 4.7k, Resistor_THT:R_Axial_DIN0207_L6.3mm_D2.5mm_P7.62mm_Horizontal, symbol Device:R
- added R3: R, Resistor_THT:R_Axial_DIN0207_L6.3mm_D2.5mm_P7.62mm_Horizontal, symbol Device:R
- added U2: (no value), Package_DIP:DIP-14_W7.62mm, symbol 74xGxx:74AHCT14
- added U4: PCF8574AP, Package_DIP:DIP-16_W7.62mm, symbol Interface_Expansion:PCF8574AP
- MX1: footprint PCM_marbastlib-mx:STAB_MX_P_8u -> PCM_marbastlib-mx:STAB_MX_P_7u
- renumbered RGB_LED23 to RGB_LED10, RGB_LED28 to RGB_LED11, RGB_LED32 to RGB_LED12, RGB_LED37 to RGB_LED13, RGB_LED41 to RGB_LED14, RGB_LED45 to RGB_LED15, RGB_LED49 to RGB_LED16, RGB_LED54 to RGB_LED17, RGB_LED59 to RGB_LED18, RGB_LED62 to RGB_LED19, RGB_LED11 to RGB_LED2, RGB_LED3 to RGB_LED20, RGB_LED8 to RGB_LED21, RGB_LED13 to RGB_LED22, RGB_LED19 to RGB_LED23, RGB_LED29 to RGB_LED25, RGB_LED33 to RGB_LED26, RGB_LED38 to RGB_LED27, RGB_LED42 to RGB_LED28, RGB_LED46 to RGB_LED29, RGB_LED17 to RGB_LED3, RGB_LED50 to RGB_LED30, RGB_LED55 to RGB_LED31, RGB_LED60 to RGB_LED32, RGB_LED63 to RGB_LED33, RGB_LED4 to RGB_LED34, RGB_LED10 to RGB_LED35, RGB_LED16 to RGB_LED36, RGB_LED21 to RGB_LED37, RGB_LED26 to RGB_LED38, RGB_LED31 to RGB_LED39, RGB_LED22 to RGB_LED4, RGB_LED36 to RGB_LED40, RGB_LED40 to RGB_LED41, RGB_LED44 to RGB_LED42, RGB_LED48 to RGB_LED43, RGB_LED53 to RGB_LED44, RGB_LED58 to RGB_LED45, RGB_LED64 to RGB_LED46, RGB_LED5 to RGB_LED47, RGB_LED14 to RGB_LED48, RGB_LED20 to RGB_LED49, RGB_LED27 to RGB_LED5, RGB_LED25 to RGB_LED50, RGB_LED30 to RGB_LED51, RGB_LED34 to RGB_LED52, RGB_LED39 to RGB_LED53, RGB_LED43 to RGB_LED54, RGB_LED47 to RGB_LED55, RGB_LED51 to RGB_LED56, RGB_LED56 to RGB_LED57, RGB_LED65 to RGB_LED58, RGB_LED6 to RGB_LED59, RGB_LED2 to RGB_LED6, RGB_LED9 to RGB_LED60, RGB_LED15 to RGB_LED61, RGB_LED35 to RGB_LED62, RGB_LED52 to RGB_LED63, RGB_LED57 to RGB_LED64, RGB_LED61 to RGB_LED65, RGB_LED12 to RGB_LED8, RGB_LED18 to RGB_LED9
Connections:
- net +3V3: now also R2.1, R3.2, U4.16 (VDD)
- net +5V: now also U2. (4Y)
- net C11: now also U4.9 (P4)
- net GND: now also U2. (4Y), U4.1 (A0), U4.2 (A1), U4.3 (A2), U4.8 (GND)
- net RE1BUTTON: now also U4.4 (P0)
- net RE2_BUTTON: now also U4.5 (P1)
- net RGB Data: now also U2. (4Y); no longer R1.1
- net SDA: now also A1.1 (GPIO0), R2.2, U4.15 (SDA); no longer A1.2 (GPIO1)
- net SPST1: now also U4.6 (P2)
- net SPST2: now also U4.7 (P3)
- net SCK renamed SCL
- net SCL: now also A1.2 (GPIO1), R3.1, U4.14 (SCL); no longer A1.1 (GPIO0)
- new net: R1.1, U2. (4Y)
- no-connect marks 19 -> 10
Other:
- moved on the sheet: C1

Commit message: reolacing files
Connections:
- net C11: now also A1.19 (GPIO14); no longer U4.9 (P4)
- net C13: now also U4.9 (P4); no longer A1.19 (GPIO14)
Changed lines of the file:
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@@
 	(wire
 		(pts
+			(xy 490.22 300.99) (xy 492.76 300.99)
+		)
+		(stroke
+			(width 0)
+			(type default)
+		)
+	)
+	(wire
+		(pts
 			(xy 386.08 171.45) (xy 386.08 173.99)
 		)
@@
 	(wire
 		(pts
-			(xy 510.54 317.5) (xy 516.89 317.5)
-		)
-		(stroke
-			(width 0)
-			(type default)
-		)
-	)
-	(wire
-		(pts
 			(xy 283.21 307.34) (xy 293.37 307.34)
 		)
@@
 	(wire
 		(pts
-			(xy 490.22 300.99) (xy 492.76 300.99)
-		)
-		(stroke
-			(width 0)
-			(type default)
-		)
-	)
-	(wire
-		(pts
 			(xy 151.13 138.43) (xy 151.13 161.29)
 		)
@@
 	(wire
 		(pts
+			(xy 510.54 317.5) (xy 516.89 317.5)
+		)
+		(stroke
+			(width 0)
+			(type default)
+		)
+	)
+	(wire
+		(pts
 			(xy 246.38 77.47) (xy 246.38 95.25)
 		)
@@
 	)
 	(label "C13"
-		(at 510.54 317.5 0)
+		(at 492.76 300.99 0)
 		(effects
 			(font
@@
 	)
 	(label "C11"
-		(at 492.76 300.99 0)
+		(at 510.54 317.5 0)
 		(effects
 			(font

Commit message: replacing grbs
Parts:
- removed U2: (no value), Package_DIP:DIP-14_W7.62mm, symbol 74xGxx:74AHCT14
- added U3: (no value), symbol 74xGxx:SN74AHCT125N
Connections:
- net +5V: now also U3. (3Y)
- net C11: now also A1.17 (GPIO13); no longer A1.19 (GPIO14)
- net C12: now also A1.19 (GPIO14); no longer A1.17 (GPIO13)
- net GND: now also U3. (3Y)
- net RGB Data: now also U3. (3Y)
- net at R1.1: now also U3. (3Y)
Changed lines of the file:
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@@
 		(at 490.22 303.53)
 	)
-	(bus_entry
-		(at 481.33 218.44)
-		(size 2.54 2.54)
-		(stroke
-			(width 0)
-			(type default)
-		)
-	)
 	(wire
 		(pts
@@
 	(wire
 		(pts
+			(xy 510.54 317.5) (xy 516.89 317.5)
+		)
+		(stroke
+			(width 0)
+			(type default)
+		)
+	)
+	(wire
+		(pts
 			(xy 345.44 302.26) (xy 345.44 252.73)
 		)
@@
 	(wire
 		(pts
-			(xy 510.54 314.96) (xy 516.89 314.96)
-		)
-		(stroke
-			(width 0)
-			(type default)
-		)
-	)
-	(wire
-		(pts
 			(xy 190.5 327.66) (xy 196.85 327.66)
 		)
@@
 	(wire
 		(pts
+			(xy 510.54 314.96) (xy 516.89 314.96)
+		)
+		(stroke
+			(width 0)
+			(type default)
+		)
+	)
+	(wire
+		(pts
 			(xy 25.4 240.03) (xy 15.24 240.03)
 		)
@@
 	(wire
 		(pts
-			(xy 510.54 317.5) (xy 516.89 317.5)
-		)
-		(stroke
-			(width 0)
-			(type default)
-		)
-	)
-	(wire
-		(pts
 			(xy 246.38 77.47) (xy 246.38 95.25)
 		)
@@
 	)
 	(label "C11"
-		(at 510.54 317.5 0)
+		(at 510.54 314.96 0)
 		(effects
 			(font
@@
 	)
 	(label "C12"
-		(at 510.54 314.96 0)
+		(at 510.54 317.5 0)
 		(effects
 			(font
@@
 	)
 	(symbol
-		(lib_id "74xGxx:74AHCT14")
-		(at 27.94 252.73 0)
-		(unit 1)
-		(body_style 1)
-		(exclude_from_sim no)
-		(in_bom yes)
-		(on_board yes)
-		(in_pos_files yes)
-		(dnp no)
-		(fields_autoplaced yes)
-		(property "Reference" "U2"
-			(at 27.94 250.19 0)
-			(hide yes)
-			(show_name no)
-			(do_not_autoplace no)
-			(effects
-				(font
-					(size 1.27 1.27)
-				)
-			)
-		)
-		(property "Value" ""
-			(at 27.94 252.73 0)
-			(show_name no)
-			(do_not_autoplace no)
-			(effects
-				(font
-					(size 1.27 1.27)
-				)
-			)
-		)
-		(property "Footprint" "Package_DIP:DIP-14_W7.62mm"
-			(at 27.94 252.73 0)
-			(hide yes)
-			(show_name no)
-			(do_not_autoplace no)
-			(effects
-				(font
-					(size 1.27 1.27)
-				)
-			)
-		)
-		(property "Datasheet" ""
-			(at 27.94 252.73 0)
-			(hide yes)
-			(show_name no)
-			(do_not_autoplace no)
-			(effects
-				(font
-					(size 1.27 1.27)
-				)
-			)
-		)
-		(property "Description" ""
-			(at 27.94 252.73 0)
-			(hide yes)
-			(show_name no)
-			(do_not_autoplace no)
-			(effects
-				(font
-					(size 1.27 1.27)
-				)
-			)
-		)
-		(pin ""
-		)
-		(pin ""
-		)
-		(pin ""
-		)
-		(pin ""
-		)
-		(pin ""
-		)
-		(pin ""
-		)
-		(pin ""
-		)
-		(pin ""
-		)
-		(pin ""
-		)
-		(pin ""
-		)
-		(pin ""
-		)
-		(pin ""
-		)
-		(pin ""
-		)
-		(pin ""
-		)
-		(instances
-			(project "Custom Keyboard"
-				(path "/0112a49c-87b1-4505-bf98-43d79642e5f4"
-					(reference "U2")
-					(unit 1)
-				)
-			)
-		)
-	)
-	(symbol
 		(lib_id "power:GND")
 		(at 328.93 257.81 180)
@@
 	(symbol
 		(lib_id "power:+5V")
-		(at 34.29 246.38 270)
+		(at 36.83 243.84 270)
 		(unit 1)
 		(body_style 1)
@@
 		(dnp no)
 		(property "Reference" "#PWR015"
-			(at 30.48 246.38 0)
+			(at 33.02 243.84 0)
 			(hide yes)
 			(show_name no)
@@
 		)
 		(property "Value" "+5V"
-			(at 35.56 244.602 90)
+			(at 39.116 246.634 90)
 			(show_name no)
 			(do_not_autoplace no)
@@
 		)
 		(property "Footprint" ""
-			(at 34.29 246.38 0)
+			(at 36.83 243.84 0)
 			(hide yes)
 			(show_name no)
@@
 		)
 		(property "Datasheet" ""
-			(at 34.29 246.38 0)
+			(at 36.83 243.84 0)
 			(hide yes)
 			(show_name no)
@@
 		)
 		(property "Description" "Power symbol creates a global label with name \"+5V\""
-			(at 34.29 246.38 0)
+			(at 36.83 243.84 0)
 			(hide yes)
 			(show_name no)
@@
 	(symbol
 		(lib_id "power:GND")
-		(at 21.59 261.62 270)
+		(at 21.59 259.08 270)
 		(unit 1)
 		(body_style 1)
@@
 		(fields_autoplaced yes)
 		(property "Reference" "#PWR037"
-			(at 15.24 261.62 0)
+			(at 15.24 259.08 0)
 			(hide yes)
 			(show_name no)
@@
 		)
 		(property "Value" "GND"
-			(at 17.78 261.6199 90)
+			(at 17.78 259.0799 90)
 			(show_name no)
 			(do_not_autoplace no)
@@
 		)
 		(property "Footprint" ""
-			(at 21.59 261.62 0)
+			(at 21.59 259.08 0)
 			(hide yes)
 			(show_name no)
@@
 		)
 		(property "Datasheet" ""
-			(at 21.59 261.62 0)
+			(at 21.59 259.08 0)
 			(hide yes)
 			(show_name no)
@@
 		)
 		(property "Description" "Power symbol creates a global label with name \"GND\" , ground"
-			(at 21.59 261.62 0)
+			(at 21.59 259.08 0)
 			(hide yes)
 			(show_name no)
@@
 					(unit 1)
 				)
+			)
+		)
+	)
+	(symbol
+		(lib_id "74xGxx:SN74AHCT125N")
+		(at 29.21 255.27 0)
+		(unit 1)
+		(body_style 1)
+		(exclude_from_sim no)
+		(in_bom yes)
+		(on_board yes)
+		(in_pos_files yes)
+		(dnp no)
+		(fields_autoplaced yes)
+		(property "Reference" "U3"
+			(at 29.21 252.73 0)
+			(hide yes)
+			(show_name no)
+			(do_not_autoplace no)
+			(effects
+				(font
+					(size 1.27 1.27)
+				)
+			)
+		)
+		(property "Value" ""
+			(at 29.21 255.27 0)
+			(show_name no)
+			(do_not_autoplace no)
+			(effects
+				(font
+					(size 1.27 1.27)
+				)
+			)
+		)
+		(property "Footprint" ""
+			(at 29.21 255.27 0)
+			(hide yes)
+			(show_name no)
+			(do_not_autoplace no)
+			(effects
+				(font
+					(size 1.27 1.27)
+				)
+			)
+		)
+		(property "Datasheet" ""
+			(at 29.21 255.27 0)
+			(hide yes)
+			(show_name no)
+			(do_not_autoplace no)
+			(effects
+				(font
+					(size 1.27 1.27)
+				)
+			)
+		)
+		(property "Description" ""
+			(at 29.21 255.27 0)
+			(hide yes)
+			(show_name no)
+			(do_not_autoplace no)
+			(effects
+				(font
+					(size 1.27 1.27)
+				)
+			)
+		)
+		(pin ""
+		)
+		(pin ""
+		)
+		(pin ""
+		)
+		(pin ""
+		)
+		(pin ""
+		)
+		(pin ""
+		)
+		(pin ""
+		)
+		(pin ""
+		)
+		(pin ""
+		)
+		(pin ""
+		)
+		(pin ""
+		)
+		(pin ""
+		)
+		(pin ""
+		)
+		(pin ""
+		)
+		(instances
+			(project "Custom Keyboard"
+				(path "/0112a49c-87b1-4505-bf98-43d79642e5f4"
+					(reference "U3")
+					(unit 1)
+				)

Commit message: replacing fabs agfain lol
Parts:
- removed U3: (no value), symbol 74xGxx:SN74AHCT125N
- added U2: SN74AHCT125N, symbol 74xGxx:SN74AHCT125N
Connections:
- net +5V: now also U2. (3Y)
- net C0: now also SW21.1, SW60.1, SW7.1
- net C1: now also SW2.1, SW22.1, SW35.1, SW48.1, SW61.1, SW8.1; no longer SW21.1, SW60.1, SW7.1
- net C10: now also SW17.1, SW31.1, SW44.1, SW57.1, SW64.1; no longer SW16.1, SW30.1, SW43.1, SW56.1, SW63.1
- net C11: now also SW18.1, SW32.1, SW45.1, SW65.1; no longer SW17.1, SW31.1, SW44.1, SW57.1, SW64.1
- net C12: now also SW19.1, SW33.1, SW46.1, SW58.1, SW66.1; no longer SW18.1, SW32.1, SW45.1, SW65.1
- net C2: now also SW23.1, SW3.1, SW36.1, SW49.1, SW9.1; no longer SW2.1, SW22.1, SW35.1, SW48.1, SW61.1, SW8.1
- net C3: now also SW10.1, SW24.1, SW37.1, SW4.1, SW50.1; no longer SW23.1, SW3.1, SW36.1, SW49.1, SW9.1
- net C4: now also SW11.1, SW25.1, SW38.1, SW5.1, SW51.1; no longer SW10.1, SW24.1, SW37.1, SW4.1, SW50.1
- net C5: now also SW12.1, SW26.1, SW39.1, SW52.1; no longer SW11.1, SW25.1, SW38.1, SW5.1, SW51.1
- net C6: now also SW13.1, SW27.1, SW40.1, SW53.1, SW62.1; no longer SW12.1, SW26.1, SW39.1, SW52.1
- net C7: now also SW14.1, SW28.1, SW41.1, SW54.1; no longer SW13.1, SW27.1, SW40.1, SW53.1, SW62.1
- net C8: now also SW15.1, SW29.1, SW42.1, SW55.1; no longer SW14.1, SW28.1, SW41.1, SW54.1
- net C9: now also SW16.1, SW30.1, SW43.1, SW56.1, SW63.1; no longer SW15.1, SW29.1, SW42.1, SW55.1
- net GND: now also U2. (3Y)
- net RGB Data: now also U2. (3Y)
- net at R1.1: now also U2. (3Y)
- removed net C13: SW19.1, SW33.1, SW46.1, SW58.1, SW66.1, U4.9 (P4)
- no-connect marks 10 -> 14

Commit message: plotted schematic
Parts:
- R3: value R -> 4.7k
Connections:
- net C0: no longer SW21.1, SW60.1, SW7.1
- net C2: now also SW7.1
- net C3: now also SW21.1
- net C4: now also SW60.1
- net R1: no longer D7.1 (K)
- net R2: no longer D21.1 (K)
- net R5: now also D21.1 (K), D7.1 (K)
Other:
- moved on the sheet: C1, D21, D60, D7, R1, RGB_LED1, RGB_LED10, RGB_LED11, RGB_LED12, RGB_LED13, RGB_LED14, RGB_LED15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

Commit message: update
Parts:
- added C2, C3: 0.1uF, Capacitor_THT:C_Disc_D5.0mm_W2.5mm_P5.00mm, symbol Device:C_Polarized
- TS1, TS2: footprint Connector_PinHeader_2.54mm:PinHeader_1x02_P2.54mm_Vertical -> Connector_Terminal_Blocks_Sockets:Terminal_4.8mm
Connections:
- net +3V3: now also C2.1
- net +5V: now also C3.1
- net GND: now also C2.2, C3.2
Other:
- moved on the sheet: C1, D1, D10, D11, D12, D13, D14, D15, D16, D17, D18, D19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

Commit message: Replacing fabs
Parts:
- removed SW1: SW_Push, MX_Only:MXOnly-1U-Hotswap, symbol Switch:SW_Push
- SW10, SW11, SW12, SW13, SW14, SW15, SW16, SW17, SW18, SW19, SW2, SW20, SW21, SW22, SW23, SW24, SW25, SW26, SW27, SW28, SW29, SW3, SW30, SW31, SW32, SW33, SW34, SW35, SW36, SW37, SW38, SW39, SW4, SW40, SW41, SW42, SW43, SW44, SW45, SW46, SW47, SW48, SW49, SW5, SW50, SW51, SW52, SW53, SW54, SW55, SW56, SW57, SW58, SW59, SW6, SW60, SW61, SW62, SW63, SW64, SW65, SW66, SW7, SW8, SW9: footprint MX_Only:MXOnly-1U-Hotswap -> Button_Switch_Keyboard:MX_Hotswap
- TS1, TS2: footprint Connector_Terminal_Blocks_Sockets:Terminal_4.8mm -> Button_Switch_Keyboard:KCD1_THT
Connections:
- net RGB_Out: now reaches U2. (3Y)
- net RGB_Out: now also R1.1
- net Net-(RGB_LED1-DIN): now reaches R1.2, RGB_LED1.4 (DIN)
Other:
- moved on the sheet: R1
